File: Flex/sensor_board/sensor_board.kicad_pcb (KiCad board)
At the start: 2 copper layers, 98.8 x 95.4 mm, 80 parts, among them J1 MOLEX 522071060, U1 FXL6408UMX, U2 VL53L7CXV0GC/1, U3 VL53L7CXV0GC/1, U4 VL53L7CXV0GC/1, U5 VL53L7CXV0GC/1, U6 VL53L7CXV0GC/1, U7 VL53L7CXV0GC/1, U8 VL53L7CXV0GC/1, U9 VL53L7CXV0GC/1

Commit message: Fix IOVDD pullup
Parts:
- J1: value MOLEX 522071060 -> Conn_01x10_Pin
Connections:
- R1 pad 1: VDD_Sensor -> IOVDD_Sensor
- R2 pad 1: VDD_Sensor -> IOVDD_Sensor
- R4 pad 1: VDD_Sensor -> IOVDD_Sensor
- R5 pad 1: VDD_Sensor -> IOVDD_Sensor
- U1 pad 15: VDD_Sensor -> IOVDD_Sensor
Routing:
- net VDD_Sensor: track 276.8 -> 246.9 mm, vias 10 -> 9
- net IOVDD_Sensor: track 397.2 -> 406.6 mm
- net GND: vias 110 -> 111
Other:
- board text added: "REV B 2026-09"
- board text removed: "REV A 2025-10"
