File: Flex/sensor_board/sensor_board.kicad_sch (KiCad schematic)
At the start: 7 parts, among them J1 Conn_01x10_Pin, U1 FXL6408UMX

Commit message: Fix IOVDD pullup
Connections:
- net IOVDD_Sensor: now also R1.1, R2.1, R4.1, R5.1, U1.15 (VCC)
- net VCC: no longer R1.1, R2.1, R4.1, R5.1, U1.15 (VCC)
